File: CAD Design/PCB 2.2.1.sch (EAGLE design)
At the start: 46 parts, among them U1 CC2538, U2 MAX1555, X1 32MHz, X2 FC-12M

Commit message: Correction
Correcting 2.2.1 with most current save
Connections:
- removed net GND3: U$4.GND, U$4.GND1, U$4.GND2, U$4.GND3
- removed net N$32: U$3.GND@10, U$3.GND@19, U$3.GND@24
- net GND: now also U$3.GND@10, U$3.GND@19, U$3.GND@24, U$4.GND, U$4.GND1, U$4.GND2, U$4.GND3
Changed lines of the file:
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@@
 <pinref part="GND40" gate="1" pin="GND"/>
+</segment>
+<segment>
+<pinref part="U$3" gate="G$1" pin="GND@10"/>
+<wire x1="58.42" y1="68.58" x2="58.42" y2="71.12" width="0.1524" layer="91"/>
+<wire x1="58.42" y1="71.12" x2="53.34" y2="71.12" width="0.1524" layer="91"/>
+<pinref part="U$3" gate="G$1" pin="GND@24"/>
+<wire x1="53.34" y1="71.12" x2="48.26" y2="71.12" width="0.1524" layer="91"/>
+<pinref part="U$3" gate="G$1" pin="GND@19"/>
+<wire x1="53.34" y1="68.58" x2="53.34" y2="71.12" width="0.1524" layer="91"/>
+<pinref part="GND41" gate="1" pin="GND"/>
+<junction x="48.26" y="71.12"/>
+<wire x1="48.26" y1="71.12" x2="48.26" y2="68.58" width="0.1524" layer="91"/>
+<junction x="53.34" y="71.12"/>
+</segment>
+<segment>
+<pinref part="U$4" gate="G$1" pin="GND"/>
+<pinref part="GND19" gate="1" pin="GND"/>
+<pinref part="U$4" gate="G$1" pin="GND3"/>
+<wire x1="139.7" y1="27.94" x2="139.7" y2="25.4" width="0.1524" layer="91"/>
+<pinref part="U$4" gate="G$1" pin="GND2"/>
+<junction x="139.7" y="25.4"/>
+<wire x1="139.7" y1="25.4" x2="139.7" y2="22.86" width="0.1524" layer="91"/>
+<pinref part="U$4" gate="G$1" pin="GND1"/>
+<junction x="139.7" y="22.86"/>
+<wire x1="139.7" y1="22.86" x2="139.7" y2="20.32" width="0.1524" layer="91"/>
+<junction x="139.7" y="20.32"/>
 </segment>
 </net>
@@
 <wire x1="88.9" y1="86.36" x2="88.9" y2="78.74" width="0.1524" layer="91"/>
 <junction x="88.9" y="78.74"/>
-</segment>
-</net>
-<net name="GND3" class="0">
-<segment>
-<pinref part="U$4" gate="G$1" pin="GND"/>
-<pinref part="GND19" gate="1" pin="GND"/>
-<pinref part="U$4" gate="G$1" pin="GND3"/>
-<wire x1="139.7" y1="27.94" x2="139.7" y2="25.4" width="0.1524" layer="91"/>
-<pinref part="U$4" gate="G$1" pin="GND2"/>
-<junction x="139.7" y="25.4"/>
-<wire x1="139.7" y1="25.4" x2="139.7" y2="22.86" width="0.1524" layer="91"/>
-<pinref part="U$4" gate="G$1" pin="GND1"/>
-<junction x="139.7" y="22.86"/>
-<wire x1="139.7" y1="22.86" x2="139.7" y2="20.32" width="0.1524" layer="91"/>
-<junction x="139.7" y="20.32"/>
 </segment>
 </net>
@@
 </segment>
 </net>
-<net name="N$32" class="0">
-<segment>
-<pinref part="U$3" gate="G$1" pin="GND@10"/>
-<wire x1="58.42" y1="68.58" x2="58.42" y2="71.12" width="0.1524" layer="91"/>
-<wire x1="58.42" y1="71.12" x2="53.34" y2="71.12" width="0.1524" layer="91"/>
-<pinref part="U$3" gate="G$1" pin="GND@24"/>
-<wire x1="53.34" y1="71.12" x2="48.26" y2="71.12" width="0.1524" layer="91"/>
-<pinref part="U$3" gate="G$1" pin="GND@19"/>
-<wire x1="53.34" y1="68.58" x2="53.34" y2="71.12" width="0.1524" layer="91"/>
-<pinref part="GND41" gate="1" pin="GND"/>
-<junction x="48.26" y="71.12"/>
-<wire x1="48.26" y1="71.12" x2="48.26" y2="68.58" width="0.1524" layer="91"/>
-<junction x="53.34" y="71.12"/>
-</segment>
-</net>
