File: CAD Design/Breakout Boards/cc2538Breakout.brd (EAGLE design)
At the start: 70.1 x 35.7 mm, 29 parts

Commit message: Commit for console switching
Moving latest changes to desktop
Routing:
- net I/O30: track 0.00 -> 62.2 mm, vias 0 -> 1
- net I/O28: track 0.00 -> 58.3 mm, vias 0 -> 3
- net I/O38: track 0.00 -> 46.1 mm, vias 0 -> 3
Changed lines of the file:
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@@
 <contactref element="C55" pad="2"/>
 <contactref element="C24" pad="2"/>
-<via x="30.48" y="3.175" extent="1-16" drill="0.6"/>
 <via x="24.13" y="12.065" extent="1-16" drill="0.6"/>
 <polygon width="0.254" layer="1">
@@
 <vertex x="0" y="0"/>
 </polygon>
-<wire x1="45.622" y1="14.732" x2="59.701" y2="24.511" width="0" layer="19" extent="1-16"/>
+<via x="53.975" y="14.605" extent="1-16" drill="0.6"/>
+<via x="52.705" y="30.48" extent="1-16" drill="0.6"/>
+<wire x1="52.705" y1="30.48" x2="59.701" y2="24.511" width="0" layer="19" extent="1-1"/>
 <wire x1="25.781" y1="27.598" x2="24.575" y2="26.11" width="0" layer="19" extent="1-16"/>
 <wire x1="30.825" y1="26.86" x2="30.861" y2="27.725" width="0" layer="19" extent="1-16"/>
+<wire x1="34.505" y1="14.605" x2="38.315" y2="17.145" width="0" layer="19" extent="1-1"/>
 <wire x1="28.575" y1="22.86" x2="30.825" y2="26.86" width="0" layer="19" extent="1-1"/>
 </signal>
@@
 <contactref element="U$3" pad="28"/>
 <contactref element="U$1" pad="30"/>
-<wire x1="10.639" y1="10.922" x2="32.575" y2="20.11" width="0" layer="19" extent="1-16"/>
+<wire x1="32.575" y1="20.11" x2="33.992" y2="20.11" width="0.254" layer="1"/>
+<wire x1="33.992" y1="20.11" x2="34.29" y2="19.812" width="0.254" layer="1"/>
+<wire x1="34.29" y1="19.812" x2="34.29" y2="18.034" width="0.254" layer="1"/>
+<wire x1="34.29" y1="18.034" x2="33.528" y2="17.272" width="0.254" layer="1"/>
+<via x="33.528" y="17.272" extent="1-16" drill="0.6"/>
+<wire x1="33.528" y1="17.272" x2="33.528" y2="17.018" width="0.254" layer="16"/>
+<wire x1="33.528" y1="17.018" x2="36.322" y2="14.224" width="0.254" layer="16"/>
+<via x="36.322" y="14.224" extent="1-16" drill="0.6"/>
+<wire x1="36.322" y1="14.224" x2="36.322" y2="7.366" width="0.254" layer="1"/>
+<wire x1="36.322" y1="7.366" x2="30.861" y2="1.778" width="0.254" layer="1"/>
+<wire x1="30.861" y1="1.778" x2="8.255" y2="1.778" width="0.254" layer="1"/>
+<wire x1="8.255" y1="1.778" x2="7.366" y2="2.794" width="0.254" layer="1"/>
+<wire x1="7.366" y1="2.794" x2="7.366" y2="9.906" width="0.254" layer="1"/>
+<wire x1="7.366" y1="9.906" x2="8.255" y2="10.795" width="0.254" layer="1"/>
+<via x="8.255" y="10.795" extent="1-16" drill="0.6"/>
+<wire x1="8.255" y1="10.795" x2="10.512" y2="10.795" width="0.254" layer="16"/>
+<wire x1="10.512" y1="10.795" x2="10.639" y2="10.922" width="0.254" layer="16"/>
 </signal>
 <signal name="I/O30">
 <contactref element="U$3" pad="30"/>
 <contactref element="U$1" pad="31"/>
-<wire x1="10.639" y1="9.652" x2="32.575" y2="20.61" width="0" layer="19" extent="1-16"/>
+<wire x1="32.575" y1="20.61" x2="34" y2="20.61" width="0.254" layer="1"/>
+<wire x1="34" y1="20.61" x2="34.671" y2="19.939" width="0.254" layer="1"/>
+<wire x1="34.671" y1="19.939" x2="34.671" y2="16.891" width="0.254" layer="1"/>
+<wire x1="34.671" y1="16.891" x2="37.084" y2="14.478" width="0.254" layer="1"/>
+<wire x1="37.084" y1="14.478" x2="37.084" y2="12.319" width="0.254" layer="1"/>
+<wire x1="37.084" y1="12.319" x2="36.83" y2="12.065" width="0.254" layer="1"/>
+<wire x1="36.83" y1="12.065" x2="36.83" y2="6.985" width="0.254" layer="1"/>
+<wire x1="36.83" y1="6.985" x2="30.988" y2="1.143" width="0.254" layer="1"/>
+<wire x1="30.988" y1="1.143" x2="8.001" y2="1.143" width="0.254" layer="1"/>
+<wire x1="8.001" y1="1.143" x2="6.604" y2="2.54" width="0.254" layer="1"/>
+<wire x1="6.604" y1="2.54" x2="6.604" y2="10.414" width="0.254" layer="1"/>
+<wire x1="6.604" y1="10.414" x2="6.985" y2="10.795" width="0.254" layer="1"/>
+<via x="6.985" y="10.795" extent="1-16" drill="0.6"/>
+<wire x1="6.985" y1="10.795" x2="8.128" y2="9.652" width="0.254" layer="16"/>
+<wire x1="8.128" y1="9.652" x2="10.639" y2="9.652" width="0.254" layer="16"/>
 </signal>
 <signal name="I/O32">
@@
 <contactref element="U$3" pad="38"/>
 <contactref element="U$1" pad="29"/>
-<wire x1="10.639" y1="4.572" x2="32.575" y2="19.61" width="0" layer="19" extent="1-16"/>
+<wire x1="32.575" y1="19.61" x2="33.857" y2="19.61" width="0.254" layer="1"/>
+<wire x1="33.857" y1="19.61" x2="33.909" y2="19.558" width="0.254" layer="1"/>
+<wire x1="33.909" y1="19.558" x2="33.909" y2="19.05" width="0.254" layer="1"/>
+<wire x1="33.909" y1="19.05" x2="33.401" y2="18.542" width="0.254" layer="1"/>
+<via x="33.401" y="18.542" extent="1-16" drill="0.6"/>
+<wire x1="33.401" y1="18.542" x2="31.115" y2="16.256" width="0.254" layer="16"/>
+<wire x1="31.115" y1="16.256" x2="31.115" y2="15.367" width="0.254" layer="16"/>
+<via x="31.115" y="15.367" extent="1-16" drill="0.6"/>
+<wire x1="31.115" y1="15.367" x2="31.115" y2="2.794" width="0.254" layer="1"/>
+<wire x1="31.115" y1="2.794" x2="30.607" y2="2.286" width="0.254" layer="1"/>
+<wire x1="30.607" y1="2.286" x2="9.017" y2="2.286" width="0.254" layer="1"/>
+<wire x1="9.017" y1="2.286" x2="8.255" y2="3.048" width="0.254" layer="1"/>
+<via x="8.255" y="3.048" extent="1-16" drill="0.6"/>
+<wire x1="8.255" y1="3.048" x2="8.255" y2="3.81" width="0.254" layer="16"/>
+<wire x1="8.255" y1="3.81" x2="8.89" y2="4.445" width="0.254" layer="16"/>
+<wire x1="8.89" y1="4.445" x2="10.512" y2="4.445" width="0.254" layer="16"/>
+<wire x1="10.512" y1="4.445" x2="10.639" y2="4.572" width="0.254" layer="16"/>
 </signal>
 <signal name="N$2">
